File: KittyWood_UVC_big/KittyWood_UVC_big.kicad_sch (KiCad schematic)
At the start: 3 parts, among them K1 Wiper control relay, Q1 PN2222A

Commit message: update
Other:
- note added: "UVC motion detect module"
Changed lines of the file:
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@@
     (stroke (width 0) (type solid) (color 0 0 0 0))
+  )
+  (text "UVC  motion detect module" (at 208.915 172.72 180)
+    (effects (font (size 1.27 1.27)) (justify right bottom))
   )
   (label "12V" (at 186.69 41.91 180)

Commit message: test
Parts:
- added U2: HC-SR501, HC-SR501:HC-SR501, symbol Sensor_extra:HC-SR501
- R1: footprint (none) -> Resistor_THT:R_Axial_DIN0207_L6.3mm_D2.5mm_P7.62mm_Horizontal
Connections:
- net GND: now also U2.3
- net at R1.1: now also U2.2
- net 12V renamed +5V
- net +5V: now also U2.1
Changed lines of the file:
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@@
-(kicad_sch (version 20200828) (generator eeschema)
+(kicad_sch (version 20201015) (generator eeschema)
   (page 1 1)
   (paper "A4")
-  (junction (at 186.69 57.15) (diameter 0.2591) (color 0 0 0 0))
-  (wire (pts (xy 149.86 68.58) (xy 161.29 68.58))
+  (junction (at 168.91 30.48) (diameter 0.259) (color 0 0 0 0))
+  (junction (at 186.69 57.15) (diameter 0.259) (color 0 0 0 0))
+  (wire (pts (xy 146.05 30.48) (xy 146.05 40.005))
+    (stroke (width 0) (type solid) (color 0 0 0 0))
+  )
+  (wire (pts (xy 146.05 30.48) (xy 168.91 30.48))
+    (stroke (width 0) (type solid) (color 0 0 0 0))
+  )
+  (wire (pts (xy 146.05 40.005) (xy 153.67 40.005))
+    (stroke (width 0) (type solid) (color 0 0 0 0))
+  )
+  (wire (pts (xy 146.05 43.18) (xy 146.05 68.58))
+    (stroke (width 0) (type solid) (color 0 0 0 0))
+  )
+  (wire (pts (xy 146.05 68.58) (xy 161.29 68.58))
+    (stroke (width 0) (type solid) (color 0 0 0 0))
+  )
+  (wire (pts (xy 151.765 46.355) (xy 151.765 50.165))
+    (stroke (width 0) (type solid) (color 0 0 0 0))
+  )
+  (wire (pts (xy 153.67 43.18) (xy 146.05 43.18))
+    (stroke (width 0) (type solid) (color 0 0 0 0))
+  )
+  (wire (pts (xy 153.67 46.355) (xy 151.765 46.355))
+    (stroke (width 0) (type solid) (color 0 0 0 0))
+  )
+  (wire (pts (xy 168.91 27.305) (xy 173.99 27.305))
+    (stroke (width 0) (type solid) (color 0 0 0 0))
+  )
+  (wire (pts (xy 168.91 30.48) (xy 168.91 27.305))
+    (stroke (width 0) (type solid) (color 0 0 0 0))
+  )
+  (wire (pts (xy 168.91 30.48) (xy 186.69 30.48))
     (stroke (width 0) (type solid) (color 0 0 0 0))
   )
@@
     (stroke (width 0) (type solid) (color 0 0 0 0))
   )
-  (wire (pts (xy 186.69 40.64) (xy 186.69 41.91))
+  (wire (pts (xy 173.99 27.305) (xy 173.99 26.67))
+    (stroke (width 0) (type solid) (color 0 0 0 0))
+  )
+  (wire (pts (xy 186.69 30.48) (xy 186.69 41.91))
     (stroke (width 0) (type solid) (color 0 0 0 0))
   )
@@
     (stroke (width 0) (type solid) (color 0 0 0 0))
   )
+  (wire (pts (xy 194.31 30.48) (xy 224.79 30.48))
+    (stroke (width 0) (type solid) (color 0 0 0 0))
+  )
+  (wire (pts (xy 194.31 41.91) (xy 194.31 30.48))
+    (stroke (width 0) (type solid) (color 0 0 0 0))
+  )
+  (wire (pts (xy 196.85 57.15) (xy 196.85 59.055))
+    (stroke (width 0) (type solid) (color 0 0 0 0))
+  )
+  (wire (pts (xy 196.85 59.055) (xy 216.535 59.055))
+    (stroke (width 0) (type solid) (color 0 0 0 0))
+  )
+  (wire (pts (xy 216.535 34.29) (xy 224.79 34.29))
+    (stroke (width 0) (type solid) (color 0 0 0 0))
+  )
+  (wire (pts (xy 216.535 59.055) (xy 216.535 34.29))
+    (stroke (width 0) (type solid) (color 0 0 0 0))
+  )
   (text "UVC  motion detect module" (at 208.915 172.72 180)
     (effects (font (size 1.27 1.27)) (justify right bottom))
   )
-  (label "12V" (at 186.69 41.91 180)
-    (effects (font (size 1.27 1.27)) (justify right bottom))
+  (symbol (lib_id "power:+5V") (at 173.99 26.67 0) (unit 1)
+    (in_bom yes) (on_board yes)
+    (property "Reference" "#PWR?" (id 0) (at 173.99 30.48 0)
+      (effects (font (size 1.27 1.27)) hide)
+    )
+    (property "Value" "+5V" (id 1) (at 174.3583 22.3456 0))
+    (property "Footprint" "" (id 2) (at 173.99 26.67 0)
+      (effects (font (size 1.27 1.27)) hide)
+    )
+    (property "Datasheet" "" (id 3) (at 173.99 26.67 0)
+      (effects (font (size 1.27 1.27)) hide)
+    )
+  )
+  (symbol (lib_id "power:GND") (at 151.765 50.165 0) (unit 1)
+    (in_bom yes) (on_board yes)
+    (property "Reference" "#PWR0103" (id 0) (at 151.765 56.515 0)
+      (effects (font (size 1.27 1.27)) hide)
+    )
+    (property "Value" "GND" (id 1) (at 151.8793 54.4894 0))
+    (property "Footprint" "" (id 2) (at 151.765 50.165 0)
+      (effects (font (size 1.27 1.27)) hide)
+    )
+    (property "Datasheet" "" (id 3) (at 151.765 50.165 0)
+      (effects (font (size 1.27 1.27)) hide)
+    )
   )
   (symbol (lib_id "power:GND") (at 186.69 85.725 0) (unit 1)
@@
     (property "Reference" "R1" (id 0) (at 165.1 63.3538 90))
     (property "Value" "10k" (id 1) (at 165.1 65.6525 90))
-    (property "Footprint" "" (id 2) (at 165.1 70.358 90)
+    (property "Footprint" "Resistor_THT:R_Axial_DIN0207_L6.3mm_D2.5mm_P7.62mm_Horizontal" (id 2) (at 165.1 70.358 90)
       (effects (font (size 1.27 1.27)) hide)
     )
@@
     )
   )
+  (symbol (lib_id "Sensor_extra:HC-SR501") (at 160.655 37.465 0) (unit 1)
+    (in_bom yes) (on_board yes)
+    (property "Reference" "U2" (id 0) (at 157.861 31.3498 0))
+    (property "Value" "HC-SR501" (id 1) (at 157.861 33.6485 0))
+    (property "Footprint" "HC-SR501:HC-SR501" (id 2) (at 161.29 41.275 0)
+      (effects (font (size 1.27 1.27) italic) (justify left) hide)
+    )
+    (property "Datasheet" "" (id 3) (at 160.655 38.735 0)
+      (effects (font (size 1.27 1.27)) hide)
+    )
+  )
   (symbol (lib_id "Relay:SANYOU_SRD_Form_C") (at 191.77 49.53 0) (unit 1)
     (in_bom yes) (on_board yes)
@@
     )
   )
+  (sheet_instances
+    (path "/" (page "1"))
+  )
   (symbol_instances
-    (path "/4f028930-c30f-494e-937f-a3ca5c62e0f3"
+    (path "/52444dd6-f906-4191-83d9-d1a5eb8ed9fa"
       (reference "#PWR0101") (unit 1) (value "GND") (footprint "")
+    )
+    (path "/4554a8a0-96ae-40f1-a609-5cef01822ef6"
+      (reference "#PWR0103") (unit 1) (value "GND") (footprint "")
+    )
+    (path "/a66cfa33-ede9-4e47-9487-f51db41d7cb7"
+      (reference "#PWR?") (unit 1) (value "+5V") (footprint "")
     )
     (path "/3983f31d-c08d-45ad-89fb-999d4d86e01d"
@@
     )
     (path "/07dfdc05-0292-40c1-9bdf-eb2444c0981a"
-      (reference "R1") (unit 1) (value "10k") (footprint "")
+      (reference "R1") (unit 1) (value "10k") (footprint "Resistor_THT:R_Axial_DIN0207_L6.3mm_D2.5mm_P7.62mm_Horizontal")
+    )
+    (path "/99319e35-a435-47f2-98ce-14be954f02d9"
+      (reference "U2") (unit 1) (value "HC-SR501") (footprint "HC-SR501:HC-SR501")
     )
   )
